Commit message: commit file 0330

File: assets/acu/acu.urdf (robot description, URDF)
Before this commit: robot E03, 9 links, 8 joints
Joints:
- joint joint0: limit lower=-3.14 upper=3.14 effort=0 velocity=0 -> lower=-6.28319 upper=6.28319 effort=0 velocity=0
- joint joint1: limit lower=-1.1775 upper=1.1775 effort=0 velocity=0 -> lower=-2.35619 upper=2.35619 effort=0 velocity=0
- joint joint2: limit lower=-1.31 upper=1.31 effort=0 velocity=0 -> lower=-2.61799 upper=2.61799 effort=0 velocity=0
- joint joint3: limit lower=-3.14 upper=3.14 effort=0 velocity=0 -> lower=-6.28319 upper=6.28319 effort=0 velocity=0
- joint joint4: limit lower=-1.3 upper=1.3 effort=0 velocity=0 -> lower=-2.56563 upper=2.56563 effort=0 velocity=0
- joint joint5: limit lower=-3.14 upper=3.14 effort=0 velocity=0 -> lower=-6.28319 upper=6.28319 effort=0 velocity=0
- joint joint7: limit lower=-3.14 upper=3.14 effort=0 velocity=0 -> lower=-6.28319 upper=6.28319 effort=0 velocity=0
